File: POVStick.sch (KiCad schematic (older format))
At the start: 26 parts, among them J1 ISP, J2 PixelOut, J3 SD_Card, J4 OLED, SW1 UP, SW2 DOWN, SW3 OK, SW4 CANCEL, U1 ATMEGA1284P-AU, Y1 12MHz

Commit message: - changed design over to UI connector instead of dedicated keys and OLED - added power fet to switch Vbat for LEDs - added 3V3 reg
Parts:
- removed J2: PixelOut, Pin_Headers:Pin_Header_Straight_1x03_Pitch2.54mm, symbol Conn_01x03
- removed J4: OLED, Pin_Headers:Pin_Header_Straight_1x04_Pitch2.54mm, symbol Conn_01x04
- removed SW1: UP, symbol SW_Push
- removed SW2: DOWN, symbol SW_Push
- removed SW3: OK, symbol SW_Push
- removed SW4: CANCEL, symbol SW_Push
- added C10, C9: 100n, Capacitors_SMD:C_0805, symbol C
- added C11: 1n, Capacitors_SMD:C_0805, symbol C
- added J2: LED, Pin_Headers:Pin_Header_Straight_1x02_Pitch2.54mm, symbol Conn_01x02
- added J4: UI, Pin_Headers:Pin_Header_Straight_2x04_Pitch2.54mm, symbol Conn_01x08
- added J5: POWER, Connectors_Terminal_Blocks:TerminalBlock_bornier-3_P5.08mm, symbol Conn_01x03
- added Q1: Q_NMOS_GSD, TO_SOT_Packages_SMD:TO-263-2, symbol Q_NMOS_GSD
- added Q2: Q_PMOS_GDS, TO_SOT_Packages_SMD:SOT-23, symbol Q_PMOS_GDS
- added R10, R9: 10k, Resistors_SMD:R_0805, symbol R
- added U2: AP1117-33, TO_SOT_Packages_SMD:SOT-223-3_TabPin2, symbol AP1117-33
Connections:
- net labels added: +BATT
- wire segments 84 -> 91
Other:
- moved on the sheet: J1, R5, R6, R7, R8

Commit message: idk
Parts:
- C1, C10, C11, C2, C3, C4, C5, C6, C7, C8, C9: symbol C -> Device:C
- J1: symbol Conn_01x06 -> conn:Conn_01x06
- J2: symbol Conn_01x02 -> conn:Conn_01x02
- J3: symbol SD_Card -> conn:SD_Card
- J4: symbol Conn_01x08 -> conn:Conn_01x08
- J5: symbol Conn_01x03 -> conn:Conn_01x03
- Q1: symbol Q_NMOS_GSD -> Device:Q_NMOS_GSD
- Q2: symbol Q_PMOS_GDS -> Device:Q_PMOS_GDS
- R1, R10, R2, R3, R4, R5, R6, R7, R8, R9: symbol R -> Device:R
- U1: symbol ATMEGA1284P-AU -> atmel:ATMEGA1284P-AU
- U2: symbol AP1117-33 -> regul:AP1117-33
- Y1: symbol Crystal -> Device:Crystal

Commit message: - changed SD socket - removed pull-ups - changed pinout of IO jack - routed the layout
Parts:
- removed J3: SD_Card, 10067847-001, symbol conn:SD_Card
- removed J4: UI, Pin_Headers:Pin_Header_Straight_2x04_Pitch2.54mm, symbol conn:Conn_01x08
- removed R3, R4, R5, R6, R7, R8: 10k, Resistors_SMD:R_0805, symbol Device:R
- added J3: Micro_SD_Card_Det_Hirose_DM3AT, Connector_Card:microSD_HC_Hirose_DM3D-SF, symbol Connector:Micro_SD_Card_Det_Hirose_DM3AT
- added J4: Conn_01x10_Male, Connector_PinSocket_2.54mm:PinSocket_1x10_P2.54mm_Vertical, symbol Connector:Conn_01x10_Male
- C1, C10, C11, C2, C3, C4, C5, C6, C7, C8, C9: footprint Capacitors_SMD:C_0805 -> Capacitor_SMD:C_0805_2012Metric
- J1: footprint Pin_Headers:Pin_Header_Straight_2x03_Pitch2.54mm -> Connector_PinHeader_2.54mm:PinHeader_2x03_P2.54mm_Vertical; symbol conn:Conn_01x06 -> POVStick-rescue:Conn_01x06-conn
- J2: footprint Pin_Headers:Pin_Header_Straight_1x02_Pitch2.54mm -> Connector_PinHeader_2.54mm:PinHeader_1x02_P2.54mm_Vertical; symbol conn:Conn_01x02 -> POVStick-rescue:Conn_01x02-conn
- J5: footprint Connectors_Terminal_Blocks:TerminalBlock_bornier-3_P5.08mm -> TerminalBlock:TerminalBlock_bornier-3_P5.08mm; symbol conn:Conn_01x03 -> POVStick-rescue:Conn_01x03-conn
- Q1: footprint TO_SOT_Packages_SMD:TO-263-2 -> Package_TO_SOT_SMD:SOT-23
- Q2: footprint TO_SOT_Packages_SMD:SOT-23 -> Package_TO_SOT_SMD:TO-252-2
- R1, R10, R2, R9: footprint Resistors_SMD:R_0805 -> Resistor_SMD:R_0805_2012Metric
- U1: footprint Housings_QFP:TQFP-44_10x10mm_Pitch0.8mm -> Package_QFP:LQFP-44_10x10mm_P0.8mm; symbol atmel:ATMEGA1284P-AU -> POVStick-rescue:ATMEGA1284P-AU-atmel
- U2: footprint TO_SOT_Packages_SMD:SOT-223-3_TabPin2 -> Package_TO_SOT_SMD:SOT-223-3_TabPin2; symbol regul:AP1117-33 -> POVStick-rescue:AP1117-33-regul
- Y1: footprint Crystals:Crystal_HC49-U_Vertical -> Crystal:Crystal_HC49-U_Vertical
Connections:
- net +3V3: now also J3.4 (VDD), J4.10 (Pin_10), J4.4 (Pin_4)
- net CLK: now also J4.2 (Pin_2)
- net DATA: now also J4.1 (Pin_1)
- net GND: now also J3.11 (SHIELD), J3.6 (VSS), J3.9 (DET_B), J4.3 (Pin_3), J4.5 (Pin_5)
- net at J1.1 (Pin_1), U1.1 ((PCINT13/MOSI)PB5): now also J3.3 (CMD)
- net at U1.10 ((PCINT25/TXD0)PD1): now also J4.8 (Pin_8)
- net at U1.11 ((PCINT26/RXD1/INT0)PD2): now also J4.7 (Pin_7)
- net at U1.12 ((PCINT27/TXD1/INT1)PD3): now also J4.6 (Pin_6)
- net at J1.4 (Pin_4), U1.2 ((PCINT14/MISO)PB6): now also J3.7 (DAT0)
- net at J1.3 (Pin_3), U1.3 ((PCINT15/SCK)PB7): now also J3.5 (CLK)
- net at U1.42 ((PCINT10/AIN0/INT2)PB2): now also R2.2, J3.10 (DET_A)
- net at U1.44 ((PCINT12/OC0B/~SS~)PB4): now also J3.2 (DAT3/CD)
- net at U1.9 ((PCINT24/RXD0)PD0): now also J4.9 (Pin_9)
