File: POVStick.kicad_pcb (KiCad board)
At the start: 2 copper layers, 73 x 19 mm, 25 parts, among them J1 ISP, J2 LED, J3 Micro_SD_Card_Det_Hirose_DM3AT, J4 Conn_01x10_Male, J5 POWER, Q1 Q_NMOS_GSD, Q2 Q_PMOS_GDS, U1 ATMEGA1284P-AU, U2 AP1117-33, Y1 12MHz

Commit message: - added home point - added GEBERBER to .gitignore - moved a REF - base for V1.0
Other:
- rule pad_to_mask_clearance: 0.051 -> 0.1
Changed lines of the file:
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@@
-(kicad_pcb (version 20171130) (host pcbnew "(5.0.2)-1")
+(kicad_pcb (version 20171130) (host pcbnew "(5.0.0)")
   (general
     (thickness 1.6)
@@
     (pad_size 1.524 1.524)
     (pad_drill 0.762)
-    (pad_to_mask_clearance 0.051)
+    (pad_to_mask_clearance 0.1)
     (solder_mask_min_width 0.25)
-    (aux_axis_origin 0 0)
-    (visible_elements FFFFFF7F)
+    (aux_axis_origin 105 82)
+    (visible_elements 7EFFFFFF)
     (pcbplotparams
-      (layerselection 0x010fc_ffffffff)
+      (layerselection 0x010f0_ffffffff)
       (usegerberextensions false)
       (usegerberattributes false)
@@
       (linewidth 0.100000)
       (plotframeref false)
-      (viasonmask false)
+      (viasonmask true)
       (mode 1)
-      (useauxorigin false)
+      (useauxorigin true)
       (hpglpennumber 1)
       (hpglpenspeed 20)
@@
       (plotinvisibletext false)
       (padsonsilk false)
-      (subtractmaskfromsilk false)
+      (subtractmaskfromsilk true)
       (outputformat 1)
       (mirror false)
-      (drillshape 1)
+      (drillshape 0)
       (scaleselection 1)
-      (outputdirectory ""))
+      (outputdirectory "GERBER"))
   )
   (net 0 "")
@@
     (tags capacitor)
     (attr smd)
-    (fp_text reference C11 (at -2.5 0 180) (layer F.SilkS)
+    (fp_text reference C11 (at -3 0 270) (layer F.SilkS)
       (effects (font (size 1 1) (thickness 0.15)))
     )
@@
   (segment (start 134 84) (end 135.25 85.25) (width 0.25) (layer B.Cu) (net 6))
   (segment (start 135.25 85.25) (end 147.99 85.25) (width 0.25) (layer B.Cu) (net 6))
-  (segment (start 133.53 87.15) (end 133 87.15) (width 0.25) (layer F.Cu) (net 42))
-  (segment (start 144.16 82.797919) (end 143.73707 82.374989) (width 0.25) (layer F.Cu) (net 42))
-  (segment (start 144.16 84) (end 144.16 82.797919) (width 0.25) (layer F.Cu) (net 42))
-  (segment (start 143.73707 82.374989) (end 136.125011 82.374989) (width 0.25) (layer F.Cu) (net 42))
-  (segment (start 136.125011 82.374989) (end 135.25 83.25) (width 0.25) (layer F.Cu) (net 42))
-  (segment (start 135.25 83.25) (end 135.25 85.43) (width 0.25) (layer F.Cu) (net 42))
-  (segment (start 135.25 85.43) (end 133.53 87.15) (width 0.25) (layer F.Cu) (net 42))
-  (segment (start 136.62 89) (end 141.62 84) (width 0.25) (layer F.Cu) (net 41))
-  (segment (start 134.85 89) (end 136.62 89) (width 0.25) (layer F.Cu) (net 41))
-  (segment (start 137.559002 89.8) (end 142.9 84.459002) (width 0.25) (layer F.Cu) (net 40))
-  (segment (start 134.85 89.8) (end 137.559002 89.8) (width 0.25) (layer F.Cu) (net 40))
-  (segment (start 142.9 84.459002) (end 142.9 83.540998) (width 0.25) (layer F.Cu) (net 40))
-  (segment (start 139.929999 83.150001) (end 139.08 84) (width 0.25) (layer F.Cu) (net 40))
-  (segment (start 142.9 83.540998) (end 142.184001 82.824999) (width 0.25) (layer F.Cu) (net 40))
-  (segment (start 142.184001 82.824999) (end 140.255001 82.824999) (width 0.25) (layer F.Cu) (net 40))
-  (segment (start 140.255001 82.824999) (end 139.929999 83.150001) (width 0.25) (layer F.Cu) (net 40))
-  (segment (start 133.8 90.6) (end 133.724999 90.524999) (width 0.25) (layer F.Cu) (net 43))
-  (segment (start 134.85 90.6) (end 133.8 90.6) (width 0.25) (layer F.Cu) (net 43))
-  (segment (start 136.54 84) (end 136.54 87.21) (width 0.25) (layer F.Cu) (net 43))
-  (segment (start 136.54 87.21) (end 135.75 88) (width 0.25) (layer F.Cu) (net 43))
-  (segment (start 134.224999 88) (end 133.724999 88.5) (width 0.25) (layer F.Cu) (net 43))
-  (segment (start 135.75 88) (end 134.224999 88) (width 0.25) (layer F.Cu) (net 43))
-  (segment (start 133.724999 90.524999) (end 133.724999 88.5) (width 0.25) (layer F.Cu) (net 43))
   (segment (start 131.4 99.9) (end 131.4 98.85) (width 0.25) (layer F.Cu) (net 7))
   (segment (start 131.324999 99.975001) (end 131.4 99.9) (width 0.25) (layer F.Cu) (net 7))
@@
   (segment (start 108.825 95.075) (end 106.65 95.075) (width 0.25) (layer F.Cu) (net 39))
   (segment (start 114.175011 100.425011) (end 108.825 95.075) (width 0.25) (layer F.Cu) (net 39))
+  (segment (start 137.559002 89.8) (end 142.9 84.459002) (width 0.25) (layer F.Cu) (net 40))
+  (segment (start 134.85 89.8) (end 137.559002 89.8) (width 0.25) (layer F.Cu) (net 40))
+  (segment (start 142.9 84.459002) (end 142.9 83.540998) (width 0.25) (layer F.Cu) (net 40))
+  (segment (start 139.929999 83.150001) (end 139.08 84) (width 0.25) (layer F.Cu) (net 40))
+  (segment (start 142.9 83.540998) (end 142.184001 82.824999) (width 0.25) (layer F.Cu) (net 40))
+  (segment (start 142.184001 82.824999) (end 140.255001 82.824999) (width 0.25) (layer F.Cu) (net 40))
+  (segment (start 140.255001 82.824999) (end 139.929999 83.150001) (width 0.25) (layer F.Cu) (net 40))
+  (segment (start 136.62 89) (end 141.62 84) (width 0.25) (layer F.Cu) (net 41))
+  (segment (start 134.85 89) (end 136.62 89) (width 0.25) (layer F.Cu) (net 41))
+  (segment (start 133.53 87.15) (end 133 87.15) (width 0.25) (layer F.Cu) (net 42))
+  (segment (start 144.16 82.797919) (end 143.73707 82.374989) (width 0.25) (layer F.Cu) (net 42))
+  (segment (start 144.16 84) (end 144.16 82.797919) (width 0.25) (layer F.Cu) (net 42))
+  (segment (start 143.73707 82.374989) (end 136.125011 82.374989) (width 0.25) (layer F.Cu) (net 42))
+  (segment (start 136.125011 82.374989) (end 135.25 83.25) (width 0.25) (layer F.Cu) (net 42))
+  (segment (start 135.25 83.25) (end 135.25 85.43) (width 0.25) (layer F.Cu) (net 42))
+  (segment (start 135.25 85.43) (end 133.53 87.15) (width 0.25) (layer F.Cu) (net 42))
+  (segment (start 133.8 90.6) (end 133.724999 90.524999) (width 0.25) (layer F.Cu) (net 43))
+  (segment (start 134.85 90.6) (end 133.8 90.6) (width 0.25) (layer F.Cu) (net 43))
+  (segment (start 136.54 84) (end 136.54 87.21) (width 0.25) (layer F.Cu) (net 43))
+  (segment (start 136.54 87.21) (end 135.75 88) (width 0.25) (layer F.Cu) (net 43))
+  (segment (start 134.224999 88) (end 133.724999 88.5) (width 0.25) (layer F.Cu) (net 43))
+  (segment (start 135.75 88) (end 134.224999 88) (width 0.25) (layer F.Cu) (net 43))
+  (segment (start 133.724999 90.524999) (end 133.724999 88.5) (width 0.25) (layer F.Cu) (net 43))
   (zone (net 3) (net_name GND) (layer F.Cu) (hatch edge 0.508)
     (connect_pads (clearance 0.25))
